File: wasd-keyboard.kicad_pcb (KiCad board)
At the start: 2 copper layers, 343.5 x 123 mm, 0 parts

Commit message: Set two upper rows
Parts:
- added D1: 1N4148W, Diode_SMD:D_0402_1005Metric, F.Cu at (-10.2, 27.2)
- added D10: 1N4148W, Diode_SMD:D_0402_1005Metric, F.Cu at (-230.2, 184.8)
- added D11: 1N4148W, Diode_SMD:D_0402_1005Metric, F.Cu at (-205.0, 184.8)
- added D12: 1N4148W, Diode_SMD:D_0402_1005Metric, F.Cu at (-208.2, 184.8)
- added D13: 1N4148W, Diode_SMD:D_0402_1005Metric, F.Cu at (-211.3, 184.8)
- added D14: 1N4148W, Diode_SMD:D_0402_1005Metric, F.Cu at (-214.5, 184.8)
- added D15: 1N4148W, Diode_SMD:D_0402_1005Metric, F.Cu at (-217.6, 184.8)
- added D16: 1N4148W, Diode_SMD:D_0402_1005Metric, F.Cu at (-220.7, 184.8)
- added D17: 1N4148W, Diode_SMD:D_0402_1005Metric, F.Cu at (-223.9, 184.8)
- added D18: 1N4148W, Diode_SMD:D_0402_1005Metric, F.Cu at (-267.8, 184.8)
- added D19: 1N4148W, Diode_SMD:D_0402_1005Metric, F.Cu at (-201.9, 184.8)
- added D2: 1N4148W, Diode_SMD:D_0402_1005Metric, F.Cu at (-280.4, 184.8)
- added D20: 1N4148W, Diode_SMD:D_0402_1005Metric, F.Cu at (-10.2, 41.1)
- added D21: 1N4148W, Diode_SMD:D_0402_1005Metric, F.Cu at (-7.02, 39.1)
- added D22: 1N4148W, Diode_SMD:D_0402_1005Metric, F.Cu at (-10.2, 39.1)
- added D23: 1N4148W, Diode_SMD:D_0402_1005Metric, F.Cu at (-10.2, 31.2)
- added D24: 1N4148W, Diode_SMD:D_0402_1005Metric, F.Cu at (-10.2, 37.1)
- added D25: 1N4148W, Diode_SMD:D_0402_1005Metric, F.Cu at (-3.88, 35.1)
- added D26: 1N4148W, Diode_SMD:D_0402_1005Metric, F.Cu at (-7.02, 35.1)
- added D27: 1N4148W, Diode_SMD:D_0402_1005Metric, F.Cu at (-277.3, 184.8)
- added D28: 1N4148W, Diode_SMD:D_0402_1005Metric, F.Cu at (-3.88, 33.1)
- added D29: 1N4148W, Diode_SMD:D_0402_1005Metric, F.Cu at (-7.02, 33.1)
- added D3: 1N4148W, Diode_SMD:D_0402_1005Metric, F.Cu at (-283.5, 184.8)
- added D30: 1N4148W, Diode_SMD:D_0402_1005Metric, F.Cu at (-10.2, 33.1)
- added D31: 1N4148W, Diode_SMD:D_0402_1005Metric, F.Cu at (-3.88, 31.2)
- added D32: 1N4148W, Diode_SMD:D_0402_1005Metric, F.Cu at (-7.02, 31.2)
- added D33: 1N4148W, Diode_SMD:D_0402_1005Metric, F.Cu at (-7.02, 37.1)
- added D34: 1N4148W, Diode_SMD:D_0402_1005Metric, F.Cu at (-289.8, 184.8)
- added D35: 1N4148W, Diode_SMD:D_0402_1005Metric, F.Cu at (-274.1, 184.8)
- added D36: 1N4148W, Diode_SMD:D_0402_1005Metric, F.Cu at (-255.3, 184.8)
- added D37: 1N4148W, Diode_SMD:D_0402_1005Metric, F.Cu at (-50.6, 89.8)
- added D38: 1N4148W, Diode_SMD:D_0402_1005Metric, F.Cu at (-10.2, 49.1)
- added D39: 1N4148W, Diode_SMD:D_0402_1005Metric, F.Cu at (-47.4, 85.8)
- added D4: 1N4148W, Diode_SMD:D_0402_1005Metric, F.Cu at (-286.7, 184.8)
- added D40: 1N4148W, Diode_SMD:D_0402_1005Metric, F.Cu at (-50.6, 87.8)
- added D41: 1N4148W, Diode_SMD:D_0402_1005Metric, F.Cu at (-44.3, 83.8)
- added D42: 1N4148W, Diode_SMD:D_0402_1005Metric, F.Cu at (-3.88, 39.1)
- added D43: 1N4148W, Diode_SMD:D_0402_1005Metric, F.Cu at (-3.88, 37.1)
- added D44: 1N4148W, Diode_SMD:D_0402_1005Metric, F.Cu at (-10.2, 45.1)
- added D45: 1N4148W, Diode_SMD:D_0402_1005Metric, F.Cu at (-151.7, 184.8)
- added D46: 1N4148W, Diode_SMD:D_0402_1005Metric, F.Cu at (-7.02, 41.1)
- added D47: 1N4148W, Diode_SMD:D_0402_1005Metric, F.Cu at (-50.6, 85.8)
- added D48: 1N4148W, Diode_SMD:D_0402_1005Metric, F.Cu at (-47.4, 83.8)
- added D49: 1N4148W, Diode_SMD:D_0402_1005Metric, F.Cu at (-30.4, 65.6)
- added D5: 1N4148W, Diode_SMD:D_0402_1005Metric, F.Cu at (-293.0, 184.8)
- added D50: 1N4148W, Diode_SMD:D_0402_1005Metric, F.Cu at (-27.2, 63.6)
- added D51: 1N4148W, Diode_SMD:D_0402_1005Metric, F.Cu at (-148.5, 184.8)
- added D52: 1N4148W, Diode_SMD:D_0402_1005Metric, F.Cu at (-30.4, 63.6)
- added D53: 1N4148W, Diode_SMD:D_0402_1005Metric, F.Cu at (-50.6, 83.8)
- added D54: 1N4148W, Diode_SMD:D_0402_1005Metric, F.Cu at (-7.02, 43.1)
- added D55: 1N4148W, Diode_SMD:D_0402_1005Metric, F.Cu at (-264.7, 184.8)
- added D56: 1N4148W, Diode_SMD:D_0402_1005Metric, F.Cu at (-233.3, 184.8)
- added D57: 1N4148W, Diode_SMD:D_0402_1005Metric, F.Cu at (-236.4, 184.8)
- added D58: 1N4148W, Diode_SMD:D_0402_1005Metric, F.Cu at (-239.6, 184.8)
- added D59: 1N4148W, Diode_SMD:D_0402_1005Metric, F.Cu at (-242.7, 184.8)
- added D6: 1N4148W, Diode_SMD:D_0402_1005Metric, F.Cu at (-227.0, 184.8)
- added D60: 1N4148W, Diode_SMD:D_0402_1005Metric, F.Cu at (-245.9, 184.8)
- added D61: 1N4148W, Diode_SMD:D_0402_1005Metric, F.Cu at (-249.0, 184.8)
- added D62: 1N4148W, Diode_SMD:D_0402_1005Metric, F.Cu at (-252.1, 184.8)
- added D63: 1N4148W, Diode_SMD:D_0402_1005Metric, F.Cu at (-3.88, 43.1)
- added D64: 1N4148W, Diode_SMD:D_0402_1005Metric, F.Cu at (-258.4, 184.8)
- added D65: 1N4148W, Diode_SMD:D_0402_1005Metric, F.Cu at (-261.6, 184.8)
- added D66: 1N4148W, Diode_SMD:D_0402_1005Metric, F.Cu at (-271.0, 184.8)
- added D67: 1N4148W, Diode_SMD:D_0402_1005Metric, F.Cu at (-111.2, 164.6)
- added D68: 1N4148W, Diode_SMD:D_0402_1005Metric, F.Cu at (-154.8, 184.8)
- added D69: 1N4148W, Diode_SMD:D_0402_1005Metric, F.Cu at (-3.88, 41.1)
- added D7: 1N4148W, Diode_SMD:D_0402_1005Metric, F.Cu at (-192.5, 184.8)
- added D70: 1N4148W, Diode_SMD:D_0402_1005Metric, F.Cu at (-7.02, 45.1)
- added D71: 1N4148W, Diode_SMD:D_0402_1005Metric, F.Cu at (-10.2, 47.1)
- added D72: 1N4148W, Diode_SMD:D_0402_1005Metric, F.Cu at (-10.2, 35.1)
- added D73: 1N4148W, Diode_SMD:D_0402_1005Metric, F.Cu at (-3.88, 25.2)
- added D74: 1N4148W, Diode_SMD:D_0402_1005Metric, F.Cu at (-3.88, 23.2)
- added D75: 1N4148W, Diode_SMD:D_0402_1005Metric, F.Cu at (-189.3, 184.8)
- added D76: 1N4148W, Diode_SMD:D_0402_1005Metric, F.Cu at (-10.2, 25.2)
- added D77: 1N4148W, Diode_SMD:D_0402_1005Metric, F.Cu at (-7.02, 23.2)
- added D78: 1N4148W, Diode_SMD:D_0402_1005Metric, F.Cu at (-170.5, 184.8)
- added D79: 1N4148W, Diode_SMD:D_0402_1005Metric, F.Cu at (-10.2, 23.2)
- added D8: 1N4148W, Diode_SMD:D_0402_1005Metric, F.Cu at (-195.6, 184.8)
- added D80: 1N4148W, Diode_SMD:D_0402_1005Metric, F.Cu at (-173.6, 184.8)
- added D81: 1N4148W, Diode_SMD:D_0402_1005Metric, F.Cu at (-10.2, 43.1)
- added D82: 1N4148W, Diode_SMD:D_0402_1005Metric, F.Cu at (-179.9, 184.8)
- added D83: 1N4148W, Diode_SMD:D_0402_1005Metric, F.Cu at (-183.1, 184.8)
- added D84: 1N4148W, Diode_SMD:D_0402_1005Metric, F.Cu at (-186.2, 184.8)
- added D85: 1N4148W, Diode_SMD:D_0402_1005Metric, F.Cu at (-7.02, 25.2)
- added D86: 1N4148W, Diode_SMD:D_0402_1005Metric, F.Cu at (-157.9, 184.8)
- added D87: 1N4148W, Diode_SMD:D_0402_1005Metric, F.Cu at (-161.1, 184.8)
- added D88: 1N4148W, Diode_SMD:D_0402_1005Metric, F.Cu at (-164.2, 184.8)
- added D89: 1N4148W, Diode_SMD:D_0402_1005Metric, F.Cu at (-167.4, 184.8)
- added D9: 1N4148W, Diode_SMD:D_0402_1005Metric, F.Cu at (-198.8, 184.8)
- added D90: 1N4148W, Diode_SMD:D_0402_1005Metric, F.Cu at (-176.8, 184.8)
- added D91: 1N4148W, Diode_SMD:D_0402_1005Metric, F.Cu at (-3.88, 29.2)
- added D92: 1N4148W, Diode_SMD:D_0402_1005Metric, F.Cu at (-7.02, 29.2)
- added D93: 1N4148W, Diode_SMD:D_0402_1005Metric, F.Cu at (-10.2, 29.2)
- added D94: 1N4148W, Diode_SMD:D_0402_1005Metric, F.Cu at (-3.88, 27.2)
- added D95: 1N4148W, Diode_SMD:D_0402_1005Metric, F.Cu at (-7.02, 27.2)
- added R1: 330R, Resistor_SMD:R_0402_1005Metric, F.Cu at (-24.8, 71.6)
- added R10: 330R, Resistor_SMD:R_0402_1005Metric, F.Cu at (-24.8, 75.5)
- added R11: 330R, Resistor_SMD:R_0402_1005Metric, F.Cu at (-30.6, 77.5)
- added R12: 330R, Resistor_SMD:R_0402_1005Metric, F.Cu at (-24.8, 67.6)
- added R13: 330R, Resistor_SMD:R_0402_1005Metric, F.Cu at (-47.9, 99.7)
- added R14: 330R, Resistor_SMD:R_0402_1005Metric, F.Cu at (-50.8, 101.7)
- added R15: 330R, Resistor_SMD:R_0402_1005Metric, F.Cu at (-50.8, 103.7)
- added R16: 330R, Resistor_SMD:R_0402_1005Metric, F.Cu at (-7.25, 47.1)
- added R17: 330R, Resistor_SMD:R_0402_1005Metric, F.Cu at (-4.34, 47.1)
- added R18: 330R, Resistor_SMD:R_0402_1005Metric, F.Cu at (-7.25, 49.1)
- added R19: 330R, Resistor_SMD:R_0402_1005Metric, F.Cu at (-47.9, 95.7)
- added R2: 330R, Resistor_SMD:R_0402_1005Metric, F.Cu at (-21.9, 71.6)
- added R20: 330R, Resistor_SMD:R_0402_1005Metric, F.Cu at (-10.4, 51.1)
- added R21: 330R, Resistor_SMD:R_0402_1005Metric, F.Cu at (-7.48, 57.0)
- added R22: 330R, Resistor_SMD:R_0402_1005Metric, F.Cu at (-4.57, 51.1)
- added R23: 330R, Resistor_SMD:R_0402_1005Metric, F.Cu at (-10.4, 53.0)
- added R24: 330R, Resistor_SMD:R_0402_1005Metric, F.Cu at (-7.48, 53.0)
- added R25: 330R, Resistor_SMD:R_0402_1005Metric, F.Cu at (-4.57, 53.0)
- added R26: 330R, Resistor_SMD:R_0402_1005Metric, F.Cu at (-10.4, 55.0)
- added R27: 330R, Resistor_SMD:R_0402_1005Metric, F.Cu at (-7.48, 55.0)
- added R28: 330R, Resistor_SMD:R_0402_1005Metric, F.Cu at (-4.57, 55.0)
- added R29: 330R, Resistor_SMD:R_0402_1005Metric, F.Cu at (-10.4, 57.0)
- added R3: 330R, Resistor_SMD:R_0402_1005Metric, F.Cu at (-27.7, 77.5)
- added R30: 330R, Resistor_SMD:R_0402_1005Metric, F.Cu at (-7.48, 51.1)
- added R31: 330R, Resistor_SMD:R_0402_1005Metric, F.Cu at (-27.5, 65.6)
- added R32: 330R, Resistor_SMD:R_0402_1005Metric, F.Cu at (-12.7, 63.6)
- added R33: 330R, Resistor_SMD:R_0402_1005Metric, F.Cu at (-24.5, 65.6)
- added R34: 330R, Resistor_SMD:R_0402_1005Metric, F.Cu at (-21.6, 65.6)
- added R35: 330R, Resistor_SMD:R_0402_1005Metric, F.Cu at (-18.7, 65.6)
- added R36: 330R, Resistor_SMD:R_0402_1005Metric, F.Cu at (-15.8, 65.6)
- added R37: 330R, Resistor_SMD:R_0402_1005Metric, F.Cu at (-12.9, 65.6)
- added R38: 330R, Resistor_SMD:R_0402_1005Metric, F.Cu at (-27.7, 67.6)
- added R39: 330R, Resistor_SMD:R_0402_1005Metric, F.Cu at (-50.8, 99.7)
- added R4: 330R, Resistor_SMD:R_0402_1005Metric, F.Cu at (-30.6, 73.5)
- added R40: 330R, Resistor_SMD:R_0402_1005Metric, F.Cu at (-21.9, 67.6)
- added R41: 330R, Resistor_SMD:R_0402_1005Metric, F.Cu at (-19.0, 67.6)
- added R42: 330R, Resistor_SMD:R_0402_1005Metric, F.Cu at (-27.7, 69.6)
- added R43: 330R, Resistor_SMD:R_0402_1005Metric, F.Cu at (-4.34, 49.1)
- added R44: 330R, Resistor_SMD:R_0402_1005Metric, F.Cu at (-45.0, 95.7)
- added R45: 330R, Resistor_SMD:R_0402_1005Metric, F.Cu at (-50.8, 97.7)
- added R46: 330R, Resistor_SMD:R_0402_1005Metric, F.Cu at (-47.9, 97.7)
- added R47: 330R, Resistor_SMD:R_0402_1005Metric, F.Cu at (-45.0, 97.7)
- added R48: 330R, Resistor_SMD:R_0402_1005Metric, F.Cu at (-47.9, 93.7)
- added R49: 330R, Resistor_SMD:R_0402_1005Metric, F.Cu at (-134.0, 184.8)
- added R5: 330R, Resistor_SMD:R_0402_1005Metric, F.Cu at (-27.7, 73.5)
- added R50: 330R, Resistor_SMD:R_0402_1005Metric, F.Cu at (-136.9, 184.8)
- added R51: 330R, Resistor_SMD:R_0402_1005Metric, F.Cu at (-139.8, 184.8)
- added R52: 330R, Resistor_SMD:R_0402_1005Metric, F.Cu at (-142.7, 184.8)
- added R53: 330R, Resistor_SMD:R_0402_1005Metric, F.Cu at (-145.6, 184.8)
- added R54: 330R, Resistor_SMD:R_0402_1005Metric, F.Cu at (-24.3, 63.6)
- added R55: 330R, Resistor_SMD:R_0402_1005Metric, F.Cu at (-30.6, 69.6)
- added R56: 330R, Resistor_SMD:R_0402_1005Metric, F.Cu at (-30.6, 67.6)
- added R57: 330R, Resistor_SMD:R_0402_1005Metric, F.Cu at (-36.0, 87.8)
- added R58: 330R, Resistor_SMD:R_0402_1005Metric, F.Cu at (-41.8, 85.8)
- added R59: 330R, Resistor_SMD:R_0402_1005Metric, F.Cu at (-38.9, 83.8)
- added R6: 330R, Resistor_SMD:R_0402_1005Metric, F.Cu at (-24.8, 73.5)
- added R60: 330R, Resistor_SMD:R_0402_1005Metric, F.Cu at (-36.0, 83.8)
- added R61: 330R, Resistor_SMD:R_0402_1005Metric, F.Cu at (-38.9, 85.8)
- added R62: 330R, Resistor_SMD:R_0402_1005Metric, F.Cu at (-36.0, 85.8)
- added R63: 330R, Resistor_SMD:R_0402_1005Metric, F.Cu at (-33.1, 85.5)
- added R64: 330R, Resistor_SMD:R_0402_1005Metric, F.Cu at (-41.8, 87.8)
- added R65: 330R, Resistor_SMD:R_0402_1005Metric, F.Cu at (-38.9, 87.8)
- added R66: 330R, Resistor_SMD:R_0402_1005Metric, F.Cu at (-41.8, 89.8)
- added R67: 330R, Resistor_SMD:R_0402_1005Metric, F.Cu at (-50.8, 95.7)
- added R68: 330R, Resistor_SMD:R_0402_1005Metric, F.Cu at (-16.0, 67.6)
- added R69: 330R, Resistor_SMD:R_0402_1005Metric, F.Cu at (-21.9, 69.6)
- added R7: 330R, Resistor_SMD:R_0402_1005Metric, F.Cu at (-21.9, 73.5)
- added R70: 330R, Resistor_SMD:R_0402_1005Metric, F.Cu at (-19.0, 69.6)
- added R71: 330R, Resistor_SMD:R_0402_1005Metric, F.Cu at (-30.6, 71.6)
- added R72: 330R, Resistor_SMD:R_0402_1005Metric, F.Cu at (-27.7, 71.6)
- added R73: 330R, Resistor_SMD:R_0402_1005Metric, F.Cu at (-19.0, 71.6)
- added R74: 330R, Resistor_SMD:R_0402_1005Metric, F.Cu at (-24.8, 77.5)
- added R75: 330R, Resistor_SMD:R_0402_1005Metric, F.Cu at (-21.4, 63.6)
- added R76: 330R, Resistor_SMD:R_0402_1005Metric, F.Cu at (-30.6, 79.5)
- added R77: 330R, Resistor_SMD:R_0402_1005Metric, F.Cu at (-27.7, 79.5)
- added R78: 330R, Resistor_SMD:R_0402_1005Metric, F.Cu at (-30.6, 81.5)
- added R79: 330R, Resistor_SMD:R_0402_1005Metric, F.Cu at (-30.6, 83.5)
- added R8: 330R, Resistor_SMD:R_0402_1005Metric, F.Cu at (-24.8, 69.6)
- added R80: 330R, Resistor_SMD:R_0402_1005Metric, F.Cu at (-47.7, 87.8)
- added R81: 330R, Resistor_SMD:R_0402_1005Metric, F.Cu at (-30.6, 75.5)
- added R82: 330R, Resistor_SMD:R_0402_1005Metric, F.Cu at (-15.6, 63.6)
- added R83: 330R, Resistor_SMD:R_0402_1005Metric, F.Cu at (-18.5, 63.6)
- added R84: 330R, Resistor_SMD:R_0402_1005Metric, F.Cu at (-47.7, 89.8)
- added R85: 330R, Resistor_SMD:R_0402_1005Metric, F.Cu at (-44.7, 89.8)
- added R86: 330R, Resistor_SMD:R_0402_1005Metric, F.Cu at (-44.7, 87.8)
- added R87: 330R, Resistor_SMD:R_0402_1005Metric, F.Cu at (-38.9, 89.8)
- added R88: 330R, Resistor_SMD:R_0402_1005Metric, F.Cu at (-50.8, 91.8)
- added R89: 330R, Resistor_SMD:R_0402_1005Metric, F.Cu at (-47.9, 91.8)
- added R9: 330R, Resistor_SMD:R_0402_1005Metric, F.Cu at (-27.7, 75.5)
- added R90: 330R, Resistor_SMD:R_0402_1005Metric, F.Cu at (-45.0, 91.8)
- added R91: 330R, Resistor_SMD:R_0402_1005Metric, F.Cu at (-42.1, 91.8)
- added R92: 330R, Resistor_SMD:R_0402_1005Metric, F.Cu at (-39.2, 91.8)
- added R93: 330R, Resistor_SMD:R_0402_1005Metric, F.Cu at (-42.1, 93.7)
- added R94: 330R, Resistor_SMD:R_0402_1005Metric, F.Cu at (-50.8, 93.7)
- added R95: 330R, Resistor_SMD:R_0402_1005Metric, F.Cu at (-45.0, 93.7)
- added SW1: Switch, Button_Switch_Keyboard:SW_Cherry_MX_1.00u_PCB_LED, F.Cu at (57.5, 117.0)
- added SW10: Switch, Button_Switch_Keyboard:SW_Cherry_MX_1.00u_PCB_LED, F.Cu at (238.0, 117.0)
- added SW11: Switch, Button_Switch_Keyboard:SW_Cherry_MX_1.00u_PCB_LED, F.Cu at (266.5, 117.0)
- added SW12: Switch, Button_Switch_Keyboard:SW_Cherry_MX_1.00u_PCB_LED, F.Cu at (285.5, 117.0)
- added SW13: Switch, Button_Switch_Keyboard:SW_Cherry_MX_1.00u_PCB_LED, F.Cu at (304.5, 117.0)
- added SW14: Switch, Button_Switch_Keyboard:SW_Cherry_MX_1.00u_PCB_LED, F.Cu at (323.5, 117.0)
- added SW15: Switch, Button_Switch_Keyboard:SW_Cherry_MX_1.00u_PCB_LED, F.Cu at (346.9, 117.0)
- added SW16: Switch, Button_Switch_Keyboard:SW_Cherry_MX_1.00u_PCB_LED, F.Cu at (365.9, 117.0)
- added SW17: Switch, Button_Switch_Keyboard:SW_Cherry_MX_1.00u_PCB_LED, F.Cu at (384.9, 117.0)
- added SW18: Switch, Button_Switch_Keyboard:SW_Cherry_MX_1.00u_PCB_LED, F.Cu at (57.5, 143.3)
- added SW19: Switch, Button_Switch_Keyboard:SW_Cherry_MX_1.00u_PCB_LED, F.Cu at (76.5, 143.3)
- added SW2: Switch, Button_Switch_Keyboard:SW_Cherry_MX_1.00u_PCB_LED, F.Cu at (76.5, 117.0)
- added SW20: Switch, Button_Switch_Keyboard:SW_Cherry_MX_1.00u_PCB_LED, F.Cu at (95.5, 143.3)
- added SW21: Switch, Button_Switch_Keyboard:SW_Cherry_MX_1.00u_PCB_LED, F.Cu at (114.5, 143.3)
- added SW22: Switch, Button_Switch_Keyboard:SW_Cherry_MX_1.00u_PCB_LED, F.Cu at (133.5, 143.3)
- added SW23: Switch, Button_Switch_Keyboard:SW_Cherry_MX_1.00u_PCB_LED, F.Cu at (152.5, 143.3)
- added SW24: Switch, Button_Switch_Keyboard:SW_Cherry_MX_1.00u_PCB_LED, F.Cu at (171.5, 143.3)
- added SW25: Switch, Button_Switch_Keyboard:SW_Cherry_MX_1.00u_PCB_LED, F.Cu at (190.5, 143.3)
- added SW26: Switch, Button_Switch_Keyboard:SW_Cherry_MX_1.00u_PCB_LED, F.Cu at (209.5, 143.3)
- added SW27: Switch, Button_Switch_Keyboard:SW_Cherry_MX_1.00u_PCB_LED, F.Cu at (228.5, 143.3)
- added SW28: Switch, Button_Switch_Keyboard:SW_Cherry_MX_1.00u_PCB_LED, F.Cu at (247.5, 143.3)
- added SW29: Switch, Button_Switch_Keyboard:SW_Cherry_MX_1.00u_PCB_LED, F.Cu at (266.5, 143.3)
- added SW3: Switch, Button_Switch_Keyboard:SW_Cherry_MX_1.00u_PCB_LED, F.Cu at (95.5, 117.0)
- added SW30: Switch, Button_Switch_Keyboard:SW_Cherry_MX_1.00u_PCB_LED, F.Cu at (285.5, 143.3)
- added SW31: Switch, Button_Switch_Keyboard:SW_Cherry_MX_1.00u_PCB_LED, F.Cu at (304.5, 143.3)
- added SW32: Switch, Button_Switch_Keyboard:SW_Cherry_MX_1.00u_PCB_LED, F.Cu at (323.5, 143.3)
- added SW33: Switch, Button_Switch_Keyboard:SW_Cherry_MX_1.00u_PCB_LED, F.Cu at (346.9, 143.3)
- added SW34: Switch, Button_Switch_Keyboard:SW_Cherry_MX_1.00u_PCB_LED, F.Cu at (365.9, 143.3)
- added SW35: Switch, Button_Switch_Keyboard:SW_Cherry_MX_1.00u_PCB_LED, F.Cu at (384.9, 143.3)
- added SW36: Switch, Button_Switch_Keyboard:SW_Cherry_MX_1.00u_PCB_LED, F.Cu at (-160.8, 128.2)
- added SW37: Switch, Button_Switch_Keyboard:SW_Cherry_MX_1.00u_PCB_LED, F.Cu at (-181.0, 148.4)
- added SW38: Switch, Button_Switch_Keyboard:SW_Cherry_MX_1.00u_PCB_LED, F.Cu at (-201.2, 168.6)
- added SW39: Switch, Button_Switch_Keyboard:SW_Cherry_MX_1.00u_PCB_LED, F.Cu at (-80.0, 27.2)
- added SW4: Switch, Button_Switch_Keyboard:SW_Cherry_MX_1.00u_PCB_LED, F.Cu at (114.5, 117.0)
- added SW40: Switch, Button_Switch_Keyboard:SW_Cherry_MX_1.00u_PCB_LED, F.Cu at (-100.2, 47.4)
- added SW41: Switch, Button_Switch_Keyboard:SW_Cherry_MX_1.00u_PCB_LED, F.Cu at (-120.4, 67.6)
- added SW42: Switch, Button_Switch_Keyboard:SW_Cherry_MX_1.00u_PCB_LED, F.Cu at (-140.6, 87.8)
- added SW43: Switch, Button_Switch_Keyboard:SW_Cherry_MX_1.00u_PCB_LED, F.Cu at (-120.4, 87.8)
- added SW44: Switch, Button_Switch_Keyboard:SW_Cherry_MX_1.00u_PCB_LED, F.Cu at (-201.2, 148.4)
- added SW45: Switch, Button_Switch_Keyboard:SW_Cherry_MX_1.00u_PCB_LED, F.Cu at (-221.4, 168.6)
- added SW46: Switch, Button_Switch_Keyboard:SW_Cherry_MX_1.00u_PCB_LED, F.Cu at (-100.2, 27.2)
- added SW47: Switch, Button_Switch_Keyboard:SW_Cherry_MX_1.00u_PCB_LED, F.Cu at (-120.4, 47.4)
- added SW48: Switch, Button_Switch_Keyboard:SW_Cherry_MX_1.00u_PCB_LED, F.Cu at (-140.6, 67.6)
- added SW49: Switch, Button_Switch_Keyboard:SW_Cherry_MX_1.00u_PCB_LED, F.Cu at (-160.8, 87.8)
- added SW5: Switch, Button_Switch_Keyboard:SW_Cherry_MX_1.00u_PCB_LED, F.Cu at (133.5, 117.0)
- added SW50: Switch, Button_Switch_Keyboard:SW_Cherry_MX_1.00u_PCB_LED, F.Cu at (-181.0, 108.0)
- added SW51: Switch, Button_Switch_Keyboard:SW_Cherry_MX_1.00u_PCB_LED, F.Cu at (-221.4, 128.2)
- added SW52: Switch, Button_Switch_Keyboard:SW_Cherry_MX_1.00u_PCB_LED, F.Cu at (-201.2, 128.2)
- added SW53: Switch, Button_Switch_Keyboard:SW_Cherry_MX_1.00u_PCB_LED, F.Cu at (-261.8, 168.6)
- added SW54: Switch, Button_Switch_Keyboard:SW_Cherry_MX_1.00u_PCB_LED, F.Cu at (-241.6, 168.6)
- added SW55: Switch, Button_Switch_Keyboard:SW_Cherry_MX_1.00u_PCB_LED, F.Cu at (-120.4, 27.2)
- added SW56: Switch, Button_Switch_Keyboard:SW_Cherry_MX_1.00u_PCB_LED, F.Cu at (-140.6, 47.4)
- added SW57: Switch, Button_Switch_Keyboard:SW_Cherry_MX_1.00u_PCB_LED, F.Cu at (-160.8, 67.6)
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Other:
- board size 343.5 x 123 mm -> 347.5 x 125 mm

Commit message: TODO: ISO Enter rotation
Parts:
- added D96: 1N4148W, Diode_SMD:D_0402_1005Metric, F.Cu at (-161.9, 41.6)
- added D97: 1N4148W, Diode_SMD:D_0402_1005Metric, F.Cu at (-158.8, 41.6)
- added R96: 330R, Resistor_SMD:R_0402_1005Metric, F.Cu at (-155.9, 41.6)
- added R97: 330R, Resistor_SMD:R_0402_1005Metric, F.Cu at (-159.0, 43.6)
- added SW320: Switch, Button_Switch_Keyboard:SW_Cherry_MX_2.00u_PCB_LED_Inv, F.Cu at (314.0, 143.3)
- added SW660: Switch, Button_Switch_Keyboard:SW_Cherry_MX_ISOEnter_PCB_LED, F.Cu at (326.2, 161.6)
- added SW670: Switch, Button_Switch_Keyboard:SW_Cherry_MX_2.25u_PCB_LED_Inv, F.Cu at (69.4, 200.3)
- added SW800: Switch, Button_Switch_Keyboard:SW_Cherry_MX_2.75u_PCB_LED_Inv, F.Cu at (306.9, 200.3)
- added SW880: Switch, Button_Switch_Keyboard:SW_Cherry_MX_2.75u_PCB_LED, F.Cu at (164.4, 219.3)
- added SW96: Switch, Button_Switch_Keyboard:SW_Cherry_MX_1.00u_PCB_LED, F.Cu at (365.9, 219.3)
- added SW97: Switch, Button_Switch_Keyboard:SW_Cherry_MX_1.00u_PCB_LED, F.Cu at (384.9, 219.3)
- SW36, SW49: footprint Button_Switch_Keyboard:SW_Cherry_MX_1.00u_PCB_LED -> Button_Switch_Keyboard:SW_Cherry_MX_1.50u_PCB_LED
- SW53, SW80: footprint Button_Switch_Keyboard:SW_Cherry_MX_1.00u_PCB_LED -> Button_Switch_Keyboard:SW_Cherry_MX_1.75u_PCB_LED
- SW66: footprint Button_Switch_Keyboard:SW_Cherry_MX_1.00u_PCB_LED -> Button_Switch_Keyboard:SW_Cherry_MX_2.25u_PCB_LED_Inv
- SW84, SW85, SW86, SW89, SW90, SW91, SW92, SW93, SW94: footprint Button_Switch_Keyboard:SW_Cherry_MX_1.00u_PCB_LED -> Button_Switch_Keyboard:SW_Cherry_MX_1.25u_PCB_LED
- SW88: footprint Button_Switch_Keyboard:SW_Cherry_MX_1.00u_PCB_LED -> Button_Switch_Keyboard:SW_Cherry_MX_6.25u_PCB_LED
- moved SW82 651.9 mm to (365.9, 200.3), turned to 180 degrees
- moved SW95 638.3 mm to (346.9, 219.3), turned to 180 degrees
- moved SW94 621.9 mm to (321.1, 219.3), turned to 180 degrees
- moved SW81 615.7 mm to (346.9, 200.3), turned to 180 degrees
- moved SW83 611.1 mm to (384.9, 200.3), turned to 180 degrees
- moved SW51 588.3 mm to (365.9, 162.3), turned to 180 degrees
- moved SW52 587.1 mm to (384.9, 162.3), turned to 180 degrees
- moved SW93 585.0 mm to (297.4, 219.3), turned to 180 degrees
- moved SW80 569.2 mm to (316.4, 200.3), turned to 180 degrees
- moved SW78 554.2 mm to (271.3, 200.3), turned to 180 degrees
- moved SW92 549.9 mm to (273.7, 219.3), turned to 180 degrees
- moved SW91 548.0 mm to (250.0, 219.3), turned to 180 degrees
- moved SW66 538.0 mm to (311.6, 181.3), turned to 180 degrees
- moved SW50 530.7 mm to (346.9, 162.3), turned to 180 degrees
- moved SW76 517.9 mm to (233.3, 200.3), turned to 180 degrees
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
Commit message: PCB finished
Parts:
- added C101: 15pF, Capacitor_SMD:C_0402_1005Metric, B.Cu at (347.8, 148.8)
- added C102: 15pF, Capacitor_SMD:C_0402_1005Metric, B.Cu at (306.5, 149.2)
- added C103: 15pF, Capacitor_SMD:C_0402_1005Metric, B.Cu at (262.8, 149.2)
- added C104: 15pF, Capacitor_SMD:C_0402_1005Metric, B.Cu at (217.7, 148.9)
- added C105: 15pF, Capacitor_SMD:C_0402_1005Metric, B.Cu at (167.7, 149.1)
- added C106: 15pF, Capacitor_SMD:C_0402_1005Metric, B.Cu at (120.9, 148.8)
- added C107: 15pF, Capacitor_SMD:C_0402_1005Metric, B.Cu at (85.9, 148.9)
- added C108: 15pF, Capacitor_SMD:C_0402_1005Metric, B.Cu at (91.3, 201.6)
- added C109: 15pF, Capacitor_SMD:C_0402_1005Metric, B.Cu at (126.4, 201.6)
- added C110: 15pF, Capacitor_SMD:C_0402_1005Metric, B.Cu at (173.4, 201.5)
- added C111: 15pF, Capacitor_SMD:C_0402_1005Metric, B.Cu at (223.5, 201.5)
- added C112: 15pF, Capacitor_SMD:C_0402_1005Metric, B.Cu at (268.4, 201.5)
- added C113: 15pF, Capacitor_SMD:C_0402_1005Metric, B.Cu at (311.4, 201.5)
- added C114: 15pF, Capacitor_SMD:C_0402_1005Metric, B.Cu at (353.5, 201.6)
- added D101: WS2812B, LED_SMD:LED_WS2812B_PLCC4_5.0x5.0mm_P3.2mm, B.Cu at (352.0, 148.0)
- added D102: WS2812B, LED_SMD:LED_WS2812B_PLCC4_5.0x5.0mm_P3.2mm, B.Cu at (311.0, 148.0)
- added D103: WS2812B, LED_SMD:LED_WS2812B_PLCC4_5.0x5.0mm_P3.2mm, B.Cu at (267.0, 148.0)
- added D104: WS2812B, LED_SMD:LED_WS2812B_PLCC4_5.0x5.0mm_P3.2mm, B.Cu at (222.0, 148.0)
- added D105: WS2812B, LED_SMD:LED_WS2812B_PLCC4_5.0x5.0mm_P3.2mm, B.Cu at (172.0, 148.0)
- added D106: WS2812B, LED_SMD:LED_WS2812B_PLCC4_5.0x5.0mm_P3.2mm, B.Cu at (125.0, 148.0)
- added D107: WS2812B, LED_SMD:LED_WS2812B_PLCC4_5.0x5.0mm_P3.2mm, B.Cu at (90.0, 148.0)
- added D108: WS2812B, LED_SMD:LED_WS2812B_PLCC4_5.0x5.0mm_P3.2mm, B.Cu at (90.0, 205.0)
- added D109: WS2812B, LED_SMD:LED_WS2812B_PLCC4_5.0x5.0mm_P3.2mm, B.Cu at (125.0, 205.0)
- added D110: WS2812B, LED_SMD:LED_WS2812B_PLCC4_5.0x5.0mm_P3.2mm, B.Cu at (172.0, 205.0)
- added D111: WS2812B, LED_SMD:LED_WS2812B_PLCC4_5.0x5.0mm_P3.2mm, B.Cu at (222.0, 205.0)
- added D112: WS2812B, LED_SMD:LED_WS2812B_PLCC4_5.0x5.0mm_P3.2mm, B.Cu at (267.0, 205.0)
- added D113: WS2812B, LED_SMD:LED_WS2812B_PLCC4_5.0x5.0mm_P3.2mm, B.Cu at (310.0, 205.0)
- added D114: WS2812B, LED_SMD:LED_WS2812B_PLCC4_5.0x5.0mm_P3.2mm, B.Cu at (352.0, 205.0)
- added J1: Conn_01x32, wasd-keyboard:Noname_1x32-1MP_P1.0mm_Horizontal, B.Cu at (194.1, 124.0)
- added Q1: BC817, Package_TO_SOT_SMD:SOT-23, B.Cu at (330.0, 201.5)
- added R200: 3K3, Resistor_SMD:R_0402_1005Metric, B.Cu at (333.6, 200.5)
- D1, D10, D11, D12, D13, D14, D15, D16, D17, D18, D19, D2, D20, D21, D22, D23, D24, D25, D26, D27, D28, D29, D3, D30, D31, D32, D33, D34, D35, D36, D37, D38, D39, D4, D40, D41, D42, D43, D44, D45, D46, D47, D48, D49, D5, D50, D51, D52, D53, D54, D55, D56, D57, D58, D59, D6, D60, D61, D62, D63, D64, D65, D66, D67, D68, D69, D7, D70, D71, D72, D73, D74, D75, D76, D77, D78, D79, D8, D80, D81, D82, D83, D84, D85, D86, D87, D88, D89, D9, D90, D91, D92, D93, D94, D95, D96, D97, R1, R10, R11, R12, R13, R14, R15, R16, R17, R18, R19, R2, R20, R21, R22, R23, R24, R25, R26, R27, R28, R29, R3, R30, R31, R32, R33, R34, R35, R36, R37, R38, R39, R4, R40, R41, R42, R43, R44, R45, R46, R47, R48, R49, R5, R50, R51, R52, R53, R54, R55, R56, R57, R58, R59, R6, R60, R61, R62, R63, R64, R65, R66, R67, R68, R69, R7, R70, R71, R72, R73, R74, R75, R76, R77, R78, R79, R8, R80, R81, R82, R83, R84, R85, R86, R87, R88, R89, R9, R90, R91, R92, R93, R94, R95, R96, R97: moved to B.Cu
- SW1: value Switch -> Esc
- SW10: value Switch -> F8
- SW11: value Switch -> F9
- SW12: value Switch -> F10
- SW13: value Switch -> F11
- SW14: value Switch -> F12
- SW15: value Switch -> PrScr
- SW16: value Switch -> ScrLock
- SW17: value Switch -> Pause
- SW18: value Switch -> Tilde
- SW19: value Switch -> 1
- SW2, SW81, SW83: value Switch -> Reserved
- SW20: value Switch -> 2
- SW21: value Switch -> 3
- SW22: value Switch -> 4
- SW23: value Switch -> 5
- SW24: value Switch -> 6
- SW25: value Switch -> 7
- SW26: value Switch -> 8
- SW27: value Switch -> 9
- SW28: value Switch -> 0
- SW29: value Switch -> -
- SW3: value Switch -> F1
- SW30: value Switch -> +
- SW31: value Switch -> JIS |
- SW32: value Switch -> JIS Backspace
- SW320: value Switch -> Backspace
- SW33: value Switch -> Ins
- SW34: value Switch -> Home
- SW35: value Switch -> PgUp
- SW36: value Switch -> Tab
- SW37: value Switch -> Q
- SW38: value Switch -> W
- SW39: value Switch -> E
- SW4: value Switch -> F2
- SW40: value Switch -> R
- SW41: value Switch -> T
- SW42: value Switch -> Y
- SW43: value Switch -> U
- SW44: value Switch -> I
- SW45: value Switch -> O
- SW46: value Switch -> P
- SW47: value Switch -> [
- SW48: value Switch -> ]
- SW49: value Switch -> ANSI \
- SW5: value Switch -> F3
- SW50: value Switch -> Del
- SW51: value Switch -> End
- SW52: value Switch -> PgDown
- SW53: value Switch -> CapsLock
- SW54: value Switch -> A
- SW55: value Switch -> S
- SW56: value Switch -> D
- SW57: value Switch -> F
- SW58: value Switch -> G
- SW59: value Switch -> H
- SW6: value Switch -> F4
- SW60: value Switch -> J
- SW61: value Switch -> K
- SW62: value Switch -> L
- SW63: value Switch -> :
- SW64: value Switch -> "
- SW65: value Switch -> ISO #
- SW66: value Switch -> ANSI Enter
- SW660: value Switch -> ISO Enter; footprint Button_Switch_Keyboard:SW_Cherry_MX_ISOEnter_PCB_LED -> Button_Switch_Keyboard:SW_Cherry_MX_ISOEnter_PCB_LED_Rot
- SW67: value Switch -> ISO L_Shift
- SW670: value Switch -> ANSI L_Shift
- SW68: value Switch -> ISO \
- SW69: value Switch -> Z
- SW7: value Switch -> F5
- SW70: value Switch -> X
- SW71: value Switch -> C
- SW72: value Switch -> V
- SW73: value Switch -> B
- SW74: value Switch -> N
- SW75: value Switch -> M
- SW76: value Switch -> <
- SW77: value Switch -> >
- SW78: value Switch -> ?
- SW79: value Switch -> JIS _
- SW8: value Switch -> F6
- SW80: value Switch -> JIS R_Shift
- SW800: value Switch -> R_Shift
- SW82: value Switch -> Up
- SW84: value Switch -> L_Ctrl
- SW85: value Switch -> L_OS
- SW86: value Switch -> L_Alt
- SW87: value Switch -> JIS Mhen
- SW88: value Switch -> Space
- SW880: value Switch -> JIS Space
- SW89: value Switch -> JIS Henk
- SW9: value Switch -> F7
- SW90: value Switch -> JIS Kana
- SW91: value Switch -> R_Alt
- SW92: value Switch -> R_OS
- SW93: value Switch -> Menu
- SW94: value Switch -> R_Ctrl
- SW95: value Switch -> Left
- SW96: value Switch -> Down
- SW97: value Switch -> Right
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Connections:
- D1 pad 1: /LABEL -> /ROW0
- D10 pad 1: /LABEL -> /ROW12
- D11 pad 1: /LABEL -> /ROW13
- D12 pad 1: /LABEL -> /ROW14
- D13 pad 1: /LABEL -> /ROW1
- D14 pad 1: /LABEL -> /ROW2
- D15 pad 1: /LABEL -> /ROW3
- D16 pad 1: /LABEL -> /ROW5
- D17 pad 1: /LABEL -> /ROW6
- D18 pad 1: /LABEL -> /ROW7
- D19 pad 1: /LABEL -> /ROW9
- D2 pad 1: /LABEL -> /ROW1
- D20 pad 1: /LABEL -> /ROW10
- D21 pad 1: /LABEL -> /ROW11
- D22 pad 1: /LABEL -> /ROW13
- D23 pad 1: /LABEL -> /ROW14
- D24 pad 1: /LABEL -> /ROW15
- D25 pad 1: /LABEL -> /ROW0
- D26 pad 1: /LABEL -> /ROW2
- D27 pad 1: /LABEL -> /ROW3
- D28 pad 1: /LABEL -> /ROW4
- D29 pad 1: /LABEL -> /ROW6
- D3 pad 1: /LABEL -> /ROW2
- D30 pad 1: /LABEL -> /ROW7
- D31 pad 1: /LABEL -> /ROW8
- D32 pad 1: /LABEL -> /ROW10
- D32 pad 2: Net-(D32-Pad2) -> /32D
- D33 pad 1: /LABEL -> /ROW11
- D34 pad 1: /LABEL -> /ROW12
- D35 pad 1: /LABEL -> /ROW14
- D36 pad 1: /LABEL -> /ROW15
- D37 pad 1: /LABEL -> /ROW0
- D38 pad 1: /LABEL -> /ROW1
- D39 pad 1: /LABEL -> /ROW3
- D4 pad 1: /LABEL -> /ROW4
- D40 pad 1: /LABEL -> /ROW4
- D41 pad 1: /LABEL -> /ROW5
- D42 pad 1: /LABEL -> /ROW7
- D43 pad 1: /LABEL -> /ROW8
- D44 pad 1: /LABEL -> /ROW9
- D45 pad 1: /LABEL -> /ROW11
- D46 pad 1: /LABEL -> /ROW12
- D47 pad 1: /LABEL -> /ROW13
- D48 pad 1: /LABEL -> /ROW15
- D49 pad 1: /LABEL -> /ROW0
- D5 pad 1: /LABEL -> /ROW5
- D50 pad 1: /LABEL -> /ROW1
- D51 pad 1: /LABEL -> /ROW2
- D52 pad 1: /LABEL -> /ROW4
- D53 pad 1: /LABEL -> /ROW5
- D54 pad 1: /LABEL -> /ROW6
- D55 pad 1: /LABEL -> /ROW8
- D56 pad 1: /LABEL -> /ROW9
- D57 pad 1: /LABEL -> /ROW10
- D58 pad 1: /LABEL -> /ROW12
- D59 pad 1: /LABEL -> /ROW13
- D6 pad 1: /LABEL -> /ROW6
- D60 pad 1: /LABEL -> /ROW14
- D61 pad 1: /LABEL -> /ROW1
- D62 pad 1: /LABEL -> /ROW2
- D63 pad 1: /LABEL -> /ROW3
- D64 pad 1: /LABEL -> /ROW5
- D65 pad 1: /LABEL -> /ROW6
- D66 pad 1: /LABEL -> /ROW7
- D66 pad 2: Net-(D66-Pad2) -> /66D
- D67 pad 1: /LABEL -> /ROW9
- D67 pad 2: Net-(D67-Pad2) -> /67D
- D68 pad 1: /LABEL -> /ROW10
- D69 pad 1: /LABEL -> /ROW11
- D7 pad 1: /LABEL -> /ROW8
- D70 pad 1: /LABEL -> /ROW13
- D71 pad 1: /LABEL -> /ROW14
- D72 pad 1: /LABEL -> /ROW15
- D73 pad 1: /LABEL -> /ROW0
- D74 pad 1: /LABEL -> /ROW2
- D75 pad 1: /LABEL -> /ROW3
- D76 pad 1: /LABEL -> /ROW4
- D77 pad 1: /LABEL -> /ROW6
- D78 pad 1: /LABEL -> /ROW7
- D79 pad 1: /LABEL -> /ROW8
- D8 pad 1: /LABEL -> /ROW9
- D80 pad 1: /LABEL -> /ROW10
- D80 pad 2: Net-(D80-Pad2) -> /80D
- D81 pad 1: /LABEL -> /ROW11
- D82 pad 1: /LABEL -> /ROW12
- D83 pad 1: /LABEL -> /ROW14
- D84 pad 1: /LABEL -> /ROW15
- D85 pad 1: /LABEL -> /ROW0
- D86 pad 1: /LABEL -> /ROW1
- D87 pad 1: /LABEL -> /ROW2
- D88 pad 1: /LABEL -> /ROW4
- D88 pad 2: Net-(D88-Pad2) -> /88D
- D89 pad 1: /LABEL -> /ROW5
- D9 pad 1: /LABEL -> /ROW10
- D90 pad 1: /LABEL -> /ROW6
- D91 pad 1: /LABEL -> /ROW7
- D92 pad 1: /LABEL -> /ROW8
- D93 pad 1: /LABEL -> /ROW10
- D94 pad 1: /LABEL -> /ROW11
- D95 pad 1: /LABEL -> /ROW12
- D96 pad 1: /LABEL -> /ROW13
- D97 pad 1: /LABEL -> /ROW14
- R1 pad 2: /LABEL -> /LED_DRV
- R10 pad 2: /LABEL -> /LED_DRV
- R11 pad 2: /LABEL -> /LED_DRV
- R12 pad 2: /LABEL -> /LED_DRV
- R13 pad 2: /LABEL -> /LED_DRV
- R14 pad 2: /LABEL -> /LED_DRV
- R15 pad 2: /LABEL -> /LED_DRV
- R16 pad 2: /LABEL -> /LED_DRV
- R17 pad 2: /LABEL -> /LED_DRV
- R18 pad 2: /LABEL -> /LED_DRV
- R19 pad 2: /LABEL -> /LED_DRV
- R2 pad 2: /LABEL -> /LED_DRV
- R20 pad 2: /LABEL -> /LED_DRV
- R21 pad 2: /LABEL -> /LED_DRV
- R22 pad 2: /LABEL -> /LED_DRV
- R23 pad 2: /LABEL -> /LED_DRV
- R24 pad 2: /LABEL -> /LED_DRV
- R25 pad 2: /LABEL -> /LED_DRV
- R26 pad 2: /LABEL -> /LED_DRV
- R27 pad 2: /LABEL -> /LED_DRV
- R28 pad 2: /LABEL -> /LED_DRV
- R29 pad 2: /LABEL -> /LED_DRV
- R3 pad 2: /LABEL -> /LED_DRV
- R30 pad 2: /LABEL -> /LED_DRV
- R31 pad 2: /LABEL -> /LED_DRV
- R32 pad 1: Net-(R32-Pad1) -> /32LED
- R32 pad 2: /LABEL -> /LED_DRV
- R33 pad 2: /LABEL -> /LED_DRV
- R34 pad 2: /LABEL -> /LED_DRV
- R35 pad 2: /LABEL -> /LED_DRV
- R36 pad 2: /LABEL -> /LED_DRV
- R37 pad 2: /LABEL -> /LED_DRV
- R38 pad 2: /LABEL -> /LED_DRV
- R39 pad 2: /LABEL -> /LED_DRV
- R4 pad 2: /LABEL -> /LED_DRV
- R40 pad 2: /LABEL -> /LED_DRV
- R41 pad 2: /LABEL -> /LED_DRV
- R42 pad 2: /LABEL -> /LED_DRV
- R43 pad 2: /LABEL -> /LED_DRV
- R44 pad 2: /LABEL -> /LED_DRV
- R45 pad 2: /LABEL -> /LED_DRV
- R46 pad 2: /LABEL -> /LED_DRV
- R47 pad 2: /LABEL -> /LED_DRV
- R48 pad 2: /LABEL -> /LED_DRV
- R49 pad 2: /LABEL -> /LED_DRV
- R5 pad 2: /LABEL -> /LED_DRV
- R50 pad 2: /LABEL -> /LED_DRV
- R51 pad 2: /LABEL -> /LED_DRV
- R52 pad 2: /LABEL -> /LED_DRV
- R53 pad 2: /LABEL -> /LED_DRV
- R54 pad 2: /LABEL -> /LED_DRV
- R55 pad 2: /LABEL -> /LED_DRV
- R56 pad 2: /LABEL -> /LED_DRV
- R57 pad 2: /LABEL -> /LED_DRV
- R58 pad 2: /LABEL -> /LED_DRV
- R59 pad 2: /LABEL -> /LED_DRV
- R6 pad 2: /LABEL -> /LED_DRV
- R60 pad 2: /LABEL -> /LED_DRV
- R61 pad 2: /LABEL -> /LED_DRV
- R62 pad 2: /LABEL -> /LED_DRV
- R63 pad 2: /LABEL -> /LED_DRV
- R64 pad 2: /LABEL -> /LED_DRV
- R65 pad 2: /LABEL -> /LED_DRV
- R66 pad 1: Net-(R66-Pad1) -> /66LED
- R66 pad 2: /LABEL -> /LED_DRV
- R67 pad 1: Net-(R67-Pad1) -> /67LED
- R67 pad 2: /LABEL -> /LED_DRV
- R68 pad 2: /LABEL -> /LED_DRV
- R69 pad 2: /LABEL -> /LED_DRV
- R7 pad 2: /LABEL -> /LED_DRV
- R70 pad 2: /LABEL -> /LED_DRV
- R71 pad 2: /LABEL -> /LED_DRV
- R72 pad 2: /LABEL -> /LED_DRV
- R73 pad 2: /LABEL -> /LED_DRV
- R74 pad 2: /LABEL -> /LED_DRV
- R75 pad 2: /LABEL -> /LED_DRV
- R76 pad 2: /LABEL -> /LED_DRV
- R77 pad 2: /LABEL -> /LED_DRV
- R78 pad 2: /LABEL -> /LED_DRV
- R79 pad 2: /LABEL -> /LED_DRV
- R8 pad 2: /LABEL -> /LED_DRV
- R80 pad 1: Net-(R80-Pad1) -> /80LED
- R80 pad 2: /LABEL -> /LED_DRV
- R81 pad 2: /LABEL -> /LED_DRV
- R82 pad 2: /LABEL -> /LED_DRV
- R83 pad 2: /LABEL -> /LED_DRV
- R84 pad 2: /LABEL -> /LED_DRV
- R85 pad 2: /LABEL -> /LED_DRV
- R86 pad 2: /LABEL -> /LED_DRV
- R87 pad 2: /LABEL -> /LED_DRV
- R88 pad 1: Net-(R88-Pad1) -> /88LED
- R88 pad 2: /LABEL -> /LED_DRV
- R89 pad 2: /LABEL -> /LED_DRV
- R9 pad 2: /LABEL -> /LED_DRV
- R90 pad 2: /LABEL -> /LED_DRV
- R91 pad 2: /LABEL -> /LED_DRV
- R92 pad 2: /LABEL -> /LED_DRV
- R93 pad 2: /LABEL -> /LED_DRV
- R94 pad 2: /LABEL -> /LED_DRV
- R95 pad 2: /LABEL -> /LED_DRV
- R96 pad 2: /LABEL -> /LED_DRV
- R97 pad 2: /LABEL -> /LED_DRV
- SW1 pad 1: /LABEL -> /COL0
- SW1 pad 4: /LABEL -> +5V
- SW10 pad 1: /LABEL -> /COL0
- SW10 pad 4: /LABEL -> +5V
- SW11 pad 1: /LABEL -> /COL0
- SW11 pad 4: /LABEL -> +5V
- SW12 pad 1: /LABEL -> /COL0
- SW12 pad 4: /LABEL -> +5V
- SW13 pad 1: /LABEL -> /COL1
- SW13 pad 4: /LABEL -> +5V
- SW14 pad 1: /LABEL -> /COL1
- SW14 pad 4: /LABEL -> +5V
- SW15 pad 1: /LABEL -> /COL1
- SW15 pad 4: /LABEL -> +5V
- SW16 pad 1: /LABEL -> /COL1
- SW16 pad 4: /LABEL -> +5V
- SW17 pad 1: /LABEL -> /COL1
- SW17 pad 4: /LABEL -> +5V
- SW18 pad 1: /LABEL -> /COL1
- SW18 pad 4: /LABEL -> +5V
- SW19 pad 1: /LABEL -> /COL1
- SW19 pad 4: /LABEL -> +5V
- SW2 pad 1: /LABEL -> /COL0
- SW2 pad 4: /LABEL -> +5V
- SW20 pad 1: /LABEL -> /COL1
- SW20 pad 4: /LABEL -> +5V
- SW21 pad 1: /LABEL -> /COL1
- SW21 pad 4: /LABEL -> +5V
- SW22 pad 1: /LABEL -> /COL1
- SW22 pad 4: /LABEL -> +5V
- SW23 pad 1: /LABEL -> /COL1
- SW23 pad 4: /LABEL -> +5V
- SW24 pad 1: /LABEL -> /COL1
- SW24 pad 4: /LABEL -> +5V
- SW25 pad 1: /LABEL -> /COL2
- SW25 pad 4: /LABEL -> +5V
- SW26 pad 1: /LABEL -> /COL2
- SW26 pad 4: /LABEL -> +5V
- SW27 pad 1: /LABEL -> /COL2
- SW27 pad 4: /LABEL -> +5V
- SW28 pad 1: /LABEL -> /COL2
- SW28 pad 4: /LABEL -> +5V
- SW29 pad 1: /LABEL -> /COL2
- SW29 pad 4: /LABEL -> +5V
- SW3 pad 1: /LABEL -> /COL0
- SW3 pad 4: /LABEL -> +5V
- SW30 pad 1: /LABEL -> /COL2
- SW30 pad 4: /LABEL -> +5V
- SW31 pad 1: /LABEL -> /COL2
- SW31 pad 4: /LABEL -> +5V
- SW32 pad 1: /LABEL -> /COL2
- SW32 pad 2: Net-(D32-Pad2) -> /32D
- SW32 pad 3: Net-(R32-Pad1) -> /32LED
- SW32 pad 4: /LABEL -> +5V
- SW320 pad 1: /LABEL -> /COL2
- SW320 pad 2: /LABEL -> /32D
- SW320 pad 3: /LABEL -> /32LED
- SW320 pad 4: /LABEL -> +5V
- SW33 pad 1: /LABEL -> /COL2
- SW33 pad 4: /LABEL -> +5V
- SW34 pad 1: /LABEL -> /COL2
- SW34 pad 4: /LABEL -> +5V
- SW35 pad 1: /LABEL -> /COL2
- SW35 pad 4: /LABEL -> +5V
- SW36 pad 1: /LABEL -> /COL2
- SW36 pad 4: /LABEL -> +5V
- SW37 pad 1: /LABEL -> /COL3
- SW37 pad 4: /LABEL -> +5V
- SW38 pad 1: /LABEL -> /COL3
- SW38 pad 4: /LABEL -> +5V
- SW39 pad 1: /LABEL -> /COL3
- SW39 pad 4: /LABEL -> +5V
- SW4 pad 1: /LABEL -> /COL0
- SW4 pad 4: /LABEL -> +5V
- SW40 pad 1: /LABEL -> /COL3
- SW40 pad 4: /LABEL -> +5V
- SW41 pad 1: /LABEL -> /COL3
- SW41 pad 4: /LABEL -> +5V
- SW42 pad 1: /LABEL -> /COL3
- SW42 pad 4: /LABEL -> +5V
- SW43 pad 1: /LABEL -> /COL3
- SW43 pad 4: /LABEL -> +5V
- SW44 pad 1: /LABEL -> /COL3
- SW44 pad 4: /LABEL -> +5V
- SW45 pad 1: /LABEL -> /COL3
- SW45 pad 4: /LABEL -> +5V
- SW46 pad 1: /LABEL -> /COL3
- SW46 pad 4: /LABEL -> +5V
- SW47 pad 1: /LABEL -> /COL3
- SW47 pad 4: /LABEL -> +5V
- SW48 pad 1: /LABEL -> /COL3
- SW48 pad 4: /LABEL -> +5V
- SW49 pad 1: /LABEL -> /COL4
- SW49 pad 4: /LABEL -> +5V
- SW5 pad 1: /LABEL -> /COL0
- SW5 pad 4: /LABEL -> +5V
- SW50 pad 1: /LABEL -> /COL4
- SW50 pad 4: /LABEL -> +5V
- SW51 pad 1: /LABEL -> /COL4
- SW51 pad 4: /LABEL -> +5V
- SW52 pad 1: /LABEL -> /COL4
- SW52 pad 4: /LABEL -> +5V
- SW53 pad 1: /LABEL -> /COL4
- SW53 pad 4: /LABEL -> +5V
- SW54 pad 1: /LABEL -> /COL4
- SW54 pad 4: /LABEL -> +5V
- SW55 pad 1: /LABEL -> /COL4
- SW55 pad 4: /LABEL -> +5V
- SW56 pad 1: /LABEL -> /COL4
- SW56 pad 4: /LABEL -> +5V
- SW57 pad 1: /LABEL -> /COL4
- SW57 pad 4: /LABEL -> +5V
- SW58 pad 1: /LABEL -> /COL4
- SW58 pad 4: /LABEL -> +5V
- SW59 pad 1: /LABEL -> /COL4
- SW59 pad 4: /LABEL -> +5V
- SW6 pad 1: /LABEL -> /COL0
- SW6 pad 4: /LABEL -> +5V
- SW60 pad 1: /LABEL -> /COL4
- SW60 pad 4: /LABEL -> +5V
- SW61 pad 1: /LABEL -> /COL5
- SW61 pad 4: /LABEL -> +5V
- SW62 pad 1: /LABEL -> /COL5
- SW62 pad 4: /LABEL -> +5V
- SW63 pad 1: /LABEL -> /COL5
- SW63 pad 4: /LABEL -> +5V
- SW64 pad 1: /LABEL -> /COL5
- SW64 pad 4: /LABEL -> +5V
- SW65 pad 1: /LABEL -> /COL5
- SW65 pad 4: /LABEL -> +5V
- SW66 pad 1: /LABEL -> /COL5
- SW66 pad 2: Net-(D66-Pad2) -> /66D
- SW66 pad 3: Net-(R66-Pad1) -> /66LED
- SW66 pad 4: /LABEL -> +5V
- SW660 pad 1: /LABEL -> /COL4
- SW660 pad 2: /LABEL -> /66D
- SW660 pad 3: /LABEL -> /66LED
- SW660 pad 4: /LABEL -> +5V
- SW67 pad 1: /LABEL -> /COL5
- SW67 pad 2: Net-(D67-Pad2) -> /67D
- SW67 pad 3: Net-(R67-Pad1) -> /67LED
- SW67 pad 4: /LABEL -> +5V
- SW670 pad 1: /LABEL -> /COL5
- SW670 pad 2: /LABEL -> /67D
- SW670 pad 3: /LABEL -> /67LED
- SW670 pad 4: /LABEL -> +5V
- SW68 pad 1: /LABEL -> /COL5
- SW68 pad 4: /LABEL -> +5V
- SW69 pad 1: /LABEL -> /COL5
- SW69 pad 4: /LABEL -> +5V
- SW7 pad 1: /LABEL -> /COL0
- SW7 pad 4: /LABEL -> +5V
- SW70 pad 1: /LABEL -> /COL5
- SW70 pad 4: /LABEL -> +5V
- SW71 pad 1: /LABEL -> /COL5
- SW71 pad 4: /LABEL -> +5V
- SW72 pad 1: /LABEL -> /COL5
- SW72 pad 4: /LABEL -> +5V
- SW73 pad 1: /LABEL -> /COL6
- SW73 pad 4: /LABEL -> +5V
- SW74 pad 1: /LABEL -> /COL6
- SW74 pad 4: /LABEL -> +5V
- SW75 pad 1: /LABEL -> /COL6
- SW75 pad 4: /LABEL -> +5V
- SW76 pad 1: /LABEL -> /COL6
- SW76 pad 4: /LABEL -> +5V
- SW77 pad 1: /LABEL -> /COL6
- SW77 pad 4: /LABEL -> +5V
- SW78 pad 1: /LABEL -> /COL6
- SW78 pad 4: /LABEL -> +5V
- SW79 pad 1: /LABEL -> /COL6
- SW79 pad 4: /LABEL -> +5V
- SW8 pad 1: /LABEL -> /COL0
- SW8 pad 4: /LABEL -> +5V
- SW80 pad 1: /LABEL -> /COL6
- SW80 pad 2: Net-(D80-Pad2) -> /80D
- SW80 pad 3: Net-(R80-Pad1) -> /80LED
- SW80 pad 4: /LABEL -> +5V
- SW800 pad 1: /LABEL -> /COL6
- SW800 pad 2: /LABEL -> /80D
- SW800 pad 3: /LABEL -> /80LED
- SW800 pad 4: /LABEL -> +5V
- SW81 pad 1: /LABEL -> /COL6
- SW81 pad 4: /LABEL -> +5V
- SW82 pad 1: /LABEL -> /COL6
- SW82 pad 4: /LABEL -> +5V
- SW83 pad 1: /LABEL -> /COL6
- SW83 pad 4: /LABEL -> +5V
- SW84 pad 1: /LABEL -> /COL6
- SW84 pad 4: /LABEL -> +5V
- SW85 pad 1: /LABEL -> /COL7
- SW85 pad 4: /LABEL -> +5V
- SW86 pad 1: /LABEL -> /COL7
- SW86 pad 4: /LABEL -> +5V
- SW87 pad 1: /LABEL -> /COL7
- SW87 pad 4: /LABEL -> +5V
- SW88 pad 1: /LABEL -> /COL7
- SW88 pad 2: Net-(D88-Pad2) -> /88D
- SW88 pad 3: Net-(R88-Pad1) -> /88LED
- SW88 pad 4: /LABEL -> +5V
- SW880 pad 1: /LABEL -> /COL7
- SW880 pad 2: /LABEL -> /88D
- SW880 pad 3: /LABEL -> /88LED
- SW880 pad 4: /LABEL -> +5V
- SW89 pad 1: /LABEL -> /COL7
- SW89 pad 4: /LABEL -> +5V
- SW9 pad 1: /LABEL -> /COL0
- SW9 pad 4: /LABEL -> +5V
- SW90 pad 1: /LABEL -> /COL7
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Routing:
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- added copper zone on B.Cu, net +5V
- added copper zone on F.Cu, net /LED_DRV
Other:
- outline, holes or cut-outs redrawn
