File: wasd-keyboard.kicad_pcb (KiCad board)
At the start: 2 copper layers, 347.5 x 125 mm, 327 parts, among them J1 Conn_01x32, Q1 BC817, SW1 Esc, SW10 F8, SW11 F9, SW12 F10, SW13 F11, SW14 F12, SW15 PrScr, SW16 ScrLock, SW17 Pause, SW18 Tilde, SW19 1, SW2 Reserved, SW20 2, SW21 3, SW22 4, SW23 5, SW24 6, SW25 7, SW26 8, SW27 9, SW28 0, SW29 -, SW3 F1, SW30 +, SW31 JIS |, SW32 JIS Backspace, SW320 Backspace, SW33 Ins, SW34 Home, SW35 PgUp, SW36 Tab, SW37 Q, SW38 W, SW39 E, SW4 F2, SW40 R, SW41 T, SW42 Y, SW43 U, SW44 I, SW45 O, SW46 P, SW47 [, SW48 ], SW49 ANSI \, SW5 F3, SW50 Del, SW51 End, SW52 PgDown, SW53 CapsLock, SW54 A, SW55 S, SW56 D, SW57 F, SW58 G, SW59 H, SW6 F4, SW60 J, SW61 K, SW62 L, SW63 :, SW64 ", SW65 ISO #, SW66 ANSI Enter, SW660 ISO Enter, SW67 ISO L_Shift, SW670 ANSI L_Shift, SW68 ISO \, SW69 Z, SW7 F5, SW70 X, SW71 C, SW72 V, SW73 B, SW74 N, SW75 M, SW76 <, SW77 >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

Commit message: Logo added
Parts:
- added G***: LOGO, wasd-keyboard:forksand, F.Cu at (375.8, 173.9)
- added G***: LOGO, wasd-keyboard:logo, F.Cu at (347.4, 175.9)
Other:
- board text added: "Copyright (C) 2019 Fork Sand, Inc. GPLv3+"

Commit message: Fixed diodes footprints, added JCSC numbers
Parts:
- removed G***: LOGO, wasd-keyboard:forksand
- removed G***: LOGO, wasd-keyboard:logo
- D1, D10, D11, D12, D13, D14, D15, D16, D17, D18, D19, D2, D20, D21, D22, D23, D24, D25, D26, D27, D28, D29, D3, D30, D31, D32, D33, D34, D35, D36, D37, D38, D39, D4, D40, D41, D42, D43, D44, D45, D46, D47, D48, D49, D5, D50, D51, D52, D53, D54, D55, D56, D57, D58, D59, D6, D60, D61, D62, D63, D64, D65, D66, D67, D68, D69, D7, D70, D71, D72, D73, D74, D75, D76, D77, D78, D79, D8, D80, D81, D82, D83, D84, D85, D86, D87, D88, D89, D9, D90, D91, D92, D93, D94, D95, D96, D97: value 1N4148W -> 1N4148WT; footprint Diode_SMD:D_0402_1005Metric -> Diode_SMD:D_SOD-523
Routing:
- net +5V: track 113.8 -> 139.9 mm, vias 35 -> 41

Commit message: Fix DRC errors
Routing:
- net /ROW6: track 696.8 -> 697.6 mm
