File: wasd-kbd80.kicad_pcb (KiCad board)
At the start: 2 copper layers, 347.5 x 125 mm, 327 parts, among them J1 Conn_01x30, Q1 BC817, SW1 Esc, SW10 F8, SW11 F9, SW12 F10, SW13 F11, SW14 F12, SW15 PrScr, SW16 ScrLock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

Commit message: Project renaming
Parts:
- added G***: LOGO, wasd-kbd80:logo, F.Cu at (347.0, 175.9)
- added G***: LOGO, wasd-kbd80:forksand, F.Cu at (375.1, 172.6)
